File: Peapod PCB.sch (KiCad schematic (older format))
At the start: 18 parts, among them J1 CONN_01X01, J2 CONN_01X02, J3 CONN_01X06, J4 CONN_01X01, J5 CONN_01X01, J6 CONN_01X01, J7 CONN_01X02, J8 CONN_01X01, U1 ESP8266

Commit message: initial plan for the outline of new peapod
Parts:
- BT1: footprint mod:Battery Mount -> Connectors_JST:JST_PH_B2B-PH-K_02x2.00mm_Straight; Manufacture Part  (none) -> B2B-PH-K-S(LF)(SN)
- J4, J8: footprint (none) -> mod:Alligator Pad
Changed lines of the file:
@@
 F 0 "BT1" H 5050 4225 50  0000 L CNN
 F 1 "Battery_Cell" H 5050 4125 50  0000 L CNN
-F 2 "mod:Battery Mount" V 4950 4185 50  0001 C CNN
+F 2 "Connectors_JST:JST_PH_B2B-PH-K_02x2.00mm_Straight" V 4950 4185 50  0001 C CNN
 F 3 "" V 4950 4185 50  0001 C CNN
+F 4 "B2B-PH-K-S(LF)(SN)" H 4950 4125 60  0001 C CNN "Manufacture Part "
 	1    4950 4125
 	1    0    0    -1
 $EndComp
 $Comp
-L GND #PWR2
+L GND #PWR01
 U 1 1 59932223
 P 4850 4225
-F 0 "#PWR2" H 4850 3975 50  0001 C CNN
+F 0 "#PWR01" H 4850 3975 50  0001 C CNN
 F 1 "GND" H 4850 4075 50  0000 C CNN
 F 2 "" H 4850 4225 50  0001 C CNN
@@
 $EndComp
 $Comp
-L GND #PWR8
+L GND #PWR02
 U 1 1 59932907
 P 6800 4100
-F 0 "#PWR8" H 6800 3850 50  0001 C CNN
+F 0 "#PWR02" H 6800 3850 50  0001 C CNN
 F 1 "GND" H 6800 3950 50  0000 C CNN
 F 2 "" H 6800 4100 50  0001 C CNN
@@
 $EndComp
 $Comp
-L GND #PWR1
+L GND #PWR03
 U 1 1 5993357D
 P 4500 3825
-F 0 "#PWR1" H 4500 3575 50  0001 C CNN
+F 0 "#PWR03" H 4500 3575 50  0001 C CNN
 F 1 "GND" H 4500 3675 50  0000 C CNN
 F 2 "" H 4500 3825 50  0001 C CNN
@@
 $EndComp
 $Comp
-L +3.3V #PWR5
+L +3.3V #PWR04
 U 1 1 59933FE4
 P 5300 3175
-F 0 "#PWR5" H 5300 3025 50  0001 C CNN
+F 0 "#PWR04" H 5300 3025 50  0001 C CNN
 F 1 "+3.3V" H 5300 3315 50  0000 C CNN
 F 2 "" H 5300 3175 50  0001 C CNN
@@
 $EndComp
 $Comp
-L +3.3V #PWR4
+L +3.3V #PWR05
 U 1 1 59934256
 P 4950 3925
-F 0 "#PWR4" H 4950 3775 50  0001 C CNN
+F 0 "#PWR05" H 4950 3775 50  0001 C CNN
 F 1 "+3.3V" H 4950 4065 50  0000 C CNN
 F 2 "" H 4950 3925 50  0001 C CNN
@@
 	4500 3775 5050 3775
 Wire Wire Line
-	4500 3475 4500 3625
-Wire Wire Line
-	4500 3625 4500 3775
-Wire Wire Line
-	4500 3775 4500 3825
+	4500 3475 4500 3825
 Connection ~ 4500 3625
 Wire Wire Line
@@
 	4950 4225 4850 4225
 Wire Wire Line
-	5125 2700 5125 2875
-Wire Wire Line
-	5125 2875 5125 3325
+	5125 2700 5125 3325
 Wire Wire Line
 	5125 2875 5325 2875
 Connection ~ 5125 2875
 Wire Wire Line
-	4825 3025 4875 3025
-Wire Wire Line
-	4875 3025 5325 3025
+	4825 3025 5325 3025
 $Comp
 L R R2
@@
 $EndComp
 Wire Wire Line
-	6625 3475 7100 3475
-Wire Wire Line
-	7100 3475 7250 3475
+	6625 3475 7250 3475
 Connection ~ 7100 3475
 $Comp
@@
 $EndComp
 $Comp
-L GND #PWR6
+L GND #PWR06
 U 1 1 599363AF
 P 5325 2700
-F 0 "#PWR6" H 5325 2450 50  0001 C CNN
+F 0 "#PWR06" H 5325 2450 50  0001 C CNN
 F 1 "GND" H 5325 2550 50  0000 C CNN
 F 2 "" H 5325 2700 50  0001 C CNN
@@
 $EndComp
 $Comp
-L +3.3V #PWR12
+L +3.3V #PWR07
 U 1 1 599466C8
 P 7100 3875
-F 0 "#PWR12" H 7100 3725 50  0001 C CNN
+F 0 "#PWR07" H 7100 3725 50  0001 C CNN
 F 1 "+3.3V" H 7100 4015 50  0000 C CNN
 F 2 "" H 7100 3875 50  0001 C CNN
@@
 	6625 3775 6800 3775
 $Comp
-L +3.3V #PWR11
+L +3.3V #PWR08
 U 1 1 59948486
 P 6975 3700
-F 0 "#PWR11" H 6975 3550 50  0001 C CNN
+F 0 "#PWR08" H 6975 3550 50  0001 C CNN
 F 1 "+3.3V" H 6975 3840 50  0000 C CNN
 F 2 "" H 6975 3700 50  0001 C CNN
@@
 	4875 2900 4875 3025
 $Comp
-L GND #PWR3
+L GND #PWR09
 U 1 1 5994872F
 P 4875 2525
-F 0 "#PWR3" H 4875 2275 50  0001 C CNN
+F 0 "#PWR09" H 4875 2275 50  0001 C CNN
 F 1 "GND" H 4875 2375 50  0000 C CNN
 F 2 "" H 4875 2525 50  0001 C CNN
@@
 	4875 2525 4875 2600
 $Comp
-L GND #PWR13
+L GND #PWR010
 U 1 1 599488CC
 P 7250 3750
-F 0 "#PWR13" H 7250 3500 50  0001 C CNN
+F 0 "#PWR010" H 7250 3500 50  0001 C CNN
 F 1 "GND" H 7250 3600 50  0000 C CNN
 F 2 "" H 7250 3750 50  0001 C CNN
@@
 $EndComp
 $Comp
-L GND #PWR7
+L GND #PWR011
 U 1 1 59948924
 P 6625 4000
-F 0 "#PWR7" H 6625 3750 50  0001 C CNN
+F 0 "#PWR011" H 6625 3750 50  0001 C CNN
 F 1 "GND" H 6625 3850 50  0000 C CNN
 F 2 "" H 6625 4000 50  0001 C CNN
@@
 $EndComp
 $Comp
-L GND #PWR10
+L GND #PWR012
 U 1 1 599480D5
 P 6875 2200
-F 0 "#PWR10" H 6875 1950 50  0001 C CNN
+F 0 "#PWR012" H 6875 1950 50  0001 C CNN
 F 1 "GND" H 6875 2050 50  0000 C CNN
 F 2 "" H 6875 2200 50  0001 C CNN
@@
 	6875 2200 7300 2200
 $Comp
-L +3.3V #PWR9
+L +3.3V #PWR013
 U 1 1 599481A2
 P 6850 2400
-F 0 "#PWR9" H 6850 2250 50  0001 C CNN
+F 0 "#PWR013" H 6850 2250 50  0001 C CNN
 F 1 "+3.3V" H 6850 2540 50  0000 C CNN
 F 2 "" H 6850 2400 50  0001 C CNN
@@
 	6850 2400 7300 2400
 Wire Wire Line
-	6625 2875 6800 2875
-Wire Wire Line
-	6800 2875 6800 2600
-Wire Wire Line
-	6800 2600 6800 2600
-Wire Wire Line
-	6800 2600 7300 2600
+	6800 2875 6625 2875
+Wire Wire Line
+	6800 2600 6800 2875
+Wire Wire Line
+	5825 2600 7300 2600
 Wire Wire Line
 	6625 3025 6625 2500
 Wire Wire Line
-	6375 2500 6625 2500
-Wire Wire Line
-	6625 2500 7300 2500
+	6375 2500 7300 2500
 NoConn ~ 7300 2700
 NoConn ~ 7300 2300
@@
 F 0 "J4" H 5825 2200 50  0000 C CNN
 F 1 "CONN_01X01" V 5925 2100 50  0000 C CNN
-F 2 "" H 5825 2100 50  0001 C CNN
+F 2 "mod:Alligator Pad" H 5825 2100 50  0001 C CNN
 F 3 "" H 5825 2100 50  0001 C CNN
 	1    5825 2100
@@
 F 0 "J8" H 6375 2200 50  0000 C CNN
 F 1 "CONN_01X01" V 6475 2100 50  0000 C CNN
-F 2 "" H 6375 2100 50  0001 C CNN
+F 2 "mod:Alligator Pad" H 6375 2100 50  0001 C CNN
 F 3 "" H 6375 2100 50  0001 C CNN
 	1    6375 2100
@@
 Connection ~ 6625 2500
 Wire Wire Line
-	6800 2600 5825 2600
-Wire Wire Line
 	5825 2600 5825 2300

Commit message: making revisions to design
Parts:
- removed J2, J7: CONN_01X02, mod:Bridge Pad, symbol CONN_01X02
- removed J3: CONN_01X06, Pin_Headers:Pin_Header_Straight_1x06_Pitch2.54mm, symbol CONN_01X06
- removed J4, J8: CONN_01X01, mod:Alligator Pad, symbol CONN_01X01
- removed R5: 10k, Resistors_SMD:R_0805_HandSoldering, symbol R
- added P1: CONN_01X08, symbol CONN_01X08
Connections:
- net +3V3: now also P1.5 (P5)
- net GND: now also U1.10 (GPIO15), P1.1 (P1), P1.3 (P3)
- net GPIO0: now reaches R4.1, U1.12 (GPIO0)
- net GPIO0: now also P1.2 (P2)
- net at U1.15 (RXD0): now also P1.6 (P6)
- net at U1.16 (TXD0): now also P1.7 (P7)
Changed lines of the file:
@@
 $EndComp
 $Comp
-L GND #PWR01
+L GND #PWR2
 U 1 1 59932223
 P 4850 4225
-F 0 "#PWR01" H 4850 3975 50  0001 C CNN
+F 0 "#PWR2" H 4850 3975 50  0001 C CNN
 F 1 "GND" H 4850 4075 50  0000 C CNN
 F 2 "" H 4850 4225 50  0001 C CNN
@@
 $EndComp
 $Comp
-L GND #PWR02
+L GND #PWR8
 U 1 1 59932907
 P 6800 4100
-F 0 "#PWR02" H 6800 3850 50  0001 C CNN
+F 0 "#PWR8" H 6800 3850 50  0001 C CNN
 F 1 "GND" H 6800 3950 50  0000 C CNN
 F 2 "" H 6800 4100 50  0001 C CNN
@@
 $EndComp
 $Comp
-L GND #PWR03
+L GND #PWR1
 U 1 1 5993357D
 P 4500 3825
-F 0 "#PWR03" H 4500 3575 50  0001 C CNN
+F 0 "#PWR1" H 4500 3575 50  0001 C CNN
 F 1 "GND" H 4500 3675 50  0000 C CNN
 F 2 "" H 4500 3825 50  0001 C CNN
@@
 $EndComp
 $Comp
-L +3.3V #PWR04
+L +3.3V #PWR5
 U 1 1 59933FE4
 P 5300 3175
-F 0 "#PWR04" H 5300 3025 50  0001 C CNN
+F 0 "#PWR5" H 5300 3025 50  0001 C CNN
 F 1 "+3.3V" H 5300 3315 50  0000 C CNN
 F 2 "" H 5300 3175 50  0001 C CNN
@@
 $EndComp
 $Comp
-L +3.3V #PWR05
+L +3.3V #PWR4
 U 1 1 59934256
 P 4950 3925
-F 0 "#PWR05" H 4950 3775 50  0001 C CNN
+F 0 "#PWR4" H 4950 3775 50  0001 C CNN
 F 1 "+3.3V" H 4950 4065 50  0000 C CNN
 F 2 "" H 4950 3925 50  0001 C CNN
@@
 Wire Wire Line
 	4950 4225 4850 4225
-Wire Wire Line
-	5125 2700 5125 3325
 Wire Wire Line
 	5125 2875 5325 2875
@@
 $EndComp
 Connection ~ 4875 3025
-$Comp
-L CONN_01X02 J7
-U 1 1 5993514F
-P 7450 3600
-F 0 "J7" H 7450 3750 50  0000 C CNN
-F 1 "CONN_01X02" V 7550 3600 50  0000 C CNN
-F 2 "mod:Bridge Pad" H 7450 3600 50  0001 C CNN
-F 3 "" H 7450 3600 50  0001 C CNN
-	1    7450 3600
-	1    0    0    -1
-$EndComp
-Wire Wire Line
-	7250 3475 7250 3550
-Wire Wire Line
-	7250 3750 7250 3650
+Wire Wire Line
+	7250 3475 7250 3700
 $Comp
 L R R4
@@
 Connection ~ 7100 3475
 $Comp
-L CONN_01X02 J2
-U 1 1 5993627D
-P 5175 2500
-F 0 "J2" H 5175 2650 50  0000 C CNN
-F 1 "CONN_01X02" V 5275 2500 50  0000 C CNN
-F 2 "mod:Bridge Pad" H 5175 2500 50  0001 C CNN
-F 3 "" H 5175 2500 50  0001 C CNN
-	1    5175 2500
-	0    -1   -1   0
-$EndComp
-$Comp
-L GND #PWR06
-U 1 1 599363AF
-P 5325 2700
-F 0 "#PWR06" H 5325 2450 50  0001 C CNN
-F 1 "GND" H 5325 2550 50  0000 C CNN
-F 2 "" H 5325 2700 50  0001 C CNN
-F 3 "" H 5325 2700 50  0001 C CNN
-	1    5325 2700
-	0    -1   -1   0
-$EndComp
-$Comp
-L +3.3V #PWR07
+L +3.3V #PWR13
 U 1 1 599466C8
 P 7100 3875
-F 0 "#PWR07" H 7100 3725 50  0001 C CNN
+F 0 "#PWR13" H 7100 3725 50  0001 C CNN
 F 1 "+3.3V" H 7100 4015 50  0000 C CNN
 F 2 "" H 7100 3875 50  0001 C CNN
@@
 	0    1    1    0
 $EndComp
-$Comp
-L R R5
-U 1 1 59946FC4
-P 6800 3925
-F 0 "R5" V 6880 3925 50  0000 C CNN
-F 1 "10k" V 6800 3925 50  0000 C CNN
-F 2 "Resistors_SMD:R_0805_HandSoldering" V 6730 3925 50  0001 C CNN
-F 3 "" H 6800 3925 50  0001 C CNN
-	1    6800 3925
-	1    0    0    -1
-$EndComp
 Wire Wire Line
 	6625 3925 6625 4000
 Wire Wire Line
-	6800 4075 6800 4100
+	6800 3775 6800 4100
 Wire Wire Line
 	6625 3775 6800 3775
 $Comp
-L +3.3V #PWR08
+L +3.3V #PWR11
 U 1 1 59948486
 P 6975 3700
-F 0 "#PWR08" H 6975 3550 50  0001 C CNN
+F 0 "#PWR11" H 6975 3550 50  0001 C CNN
 F 1 "+3.3V" H 6975 3840 50  0000 C CNN
 F 2 "" H 6975 3700 50  0001 C CNN
@@
 	4875 2900 4875 3025
 $Comp
-L GND #PWR09
+L GND #PWR3
 U 1 1 5994872F
 P 4875 2525
-F 0 "#PWR09" H 4875 2275 50  0001 C CNN
+F 0 "#PWR3" H 4875 2275 50  0001 C CNN
 F 1 "GND" H 4875 2375 50  0000 C CNN
 F 2 "" H 4875 2525 50  0001 C CNN
@@
 	4875 2525 4875 2600
 $Comp
-L GND #PWR010
+L GND #PWR12
 U 1 1 599488CC
-P 7250 3750
-F 0 "#PWR010" H 7250 3500 50  0001 C CNN
-F 1 "GND" H 7250 3600 50  0000 C CNN
-F 2 "" H 7250 3750 50  0001 C CNN
-F 3 "" H 7250 3750 50  0001 C CNN
-	1    7250 3750
-	1    0    0    -1
-$EndComp
-$Comp
-L GND #PWR011
+P 7025 1650
+F 0 "#PWR12" H 7025 1400 50  0001 C CNN
+F 1 "GND" H 7025 1500 50  0000 C CNN
+F 2 "" H 7025 1650 50  0001 C CNN
+F 3 "" H 7025 1650 50  0001 C CNN
+	1    7025 1650
+	0    1    1    0
+$EndComp
+$Comp
+L GND #PWR7
 U 1 1 59948924
 P 6625 4000
-F 0 "#PWR011" H 6625 3750 50  0001 C CNN
+F 0 "#PWR7" H 6625 3750 50  0001 C CNN
 F 1 "GND" H 6625 3850 50  0000 C CNN
 F 2 "" H 6625 4000 50  0001 C CNN
@@
 Wire Wire Line
 	5125 3325 5325 3325
-Wire Wire Line
-	5225 2700 5325 2700
 Wire Wire Line
 	4525 3025 4525 3075
@@
 	5325 3925 4950 3925
 $Comp
-L CONN_01X06 J3
-U 1 1 59947FD8
-P 7500 2450
-F 0 "J3" H 7500 2800 50  0000 C CNN
-F 1 "CONN_01X06" V 7600 2450 50  0000 C CNN
-F 2 "Pin_Headers:Pin_Header_Straight_1x06_Pitch2.54mm" H 7500 2450 50  0001 C CNN
-F 3 "" H 7500 2450 50  0001 C CNN
-	1    7500 2450
-	1    0    0    -1
-$EndComp
-$Comp
-L GND #PWR012
+L GND #PWR10
 U 1 1 599480D5
 P 6875 2200
-F 0 "#PWR012" H 6875 1950 50  0001 C CNN
+F 0 "#PWR10" H 6875 1950 50  0001 C CNN
 F 1 "GND" H 6875 2050 50  0000 C CNN
 F 2 "" H 6875 2200 50  0001 C CNN
@@
 	6875 2200 7300 2200
 $Comp
-L +3.3V #PWR013
+L +3.3V #PWR9
 U 1 1 599481A2
 P 6850 2400
-F 0 "#PWR013" H 6850 2250 50  0001 C CNN
+F 0 "#PWR9" H 6850 2250 50  0001 C CNN
 F 1 "+3.3V" H 6850 2540 50  0000 C CNN
 F 2 "" H 6850 2400 50  0001 C CNN
@@
 	6800 2600 6800 2875
 Wire Wire Line
-	5825 2600 7300 2600
-Wire Wire Line
 	6625 3025 6625 2500
-Wire Wire Line
-	6375 2500 7300 2500
 NoConn ~ 7300 2700
 NoConn ~ 7300 2300
@@
 	1    0    0    -1
 $EndComp
-$Comp
-L CONN_01X01 J4
-U 1 1 5995C3B2
-P 5825 2100
-F 0 "J4" H 5825 2200 50  0000 C CNN
-F 1 "CONN_01X01" V 5925 2100 50  0000 C CNN
-F 2 "mod:Alligator Pad" H 5825 2100 50  0001 C CNN
-F 3 "" H 5825 2100 50  0001 C CNN
-	1    5825 2100
-	0    -1   -1   0
-$EndComp
-$Comp
-L CONN_01X01 J8
-U 1 1 5995C3FF
-P 6375 2100
-F 0 "J8" H 6375 2200 50  0000 C CNN
-F 1 "CONN_01X01" V 6475 2100 50  0000 C CNN
-F 2 "mod:Alligator Pad" H 6375 2100 50  0001 C CNN
-F 3 "" H 6375 2100 50  0001 C CNN
-	1    6375 2100
-	0    -1   -1   0
-$EndComp
-Wire Wire Line
-	6375 2500 6375 2300
 Connection ~ 6625 2500
-Wire Wire Line
-	5825 2600 5825 2300
 Connection ~ 6800 2600
+Text GLabel 7325 3700 2    60   Input ~ 0
+GPIO0
+$Comp
+L CONN_01X08 P1
+U 1 1 59BC2795
+P 7500 2350
+F 0 "P1" H 7500 2800 50  0000 C CNN
+F 1 "CONN_01X08" V 7600 2350 50  0000 C CNN
+F 2 "" H 7500 2350 50  0000 C CNN
+F 3 "" H 7500 2350 50  0000 C CNN
+	1    7500 2350
+	1    0    0    -1
+$EndComp
+Text GLabel 7050 1825 0    60   Output ~ 0
+GPIO0
+Wire Wire Line
+	7300 2100 7150 2100
+Wire Wire Line
+	7150 2100 7150 1825
+Wire Wire Line
+	7150 1825 7050 1825
+Wire Wire Line
+	7300 2000 7300 1650
+Wire Wire Line
+	7300 1650 7025 1650
+Wire Wire Line
+	7250 3700 7325 3700
+Wire Wire Line
+	5125 3325 5125 2875
+Wire Wire Line
+	7300 2600 6800 2600
+Wire Wire Line
+	6625 2500 7300 2500
 $EndSCHEMATC

Commit message: final touches on peapod. Feature complete.
Parts:
- removed R3: 10k, Resistors_SMD:R_0805_HandSoldering, symbol R
- P1: footprint (none) -> Pin_Headers:Pin_Header_Straight_1x08_Pitch2.54mm
- renumbered J5 to J2, J6 to J3, R4 to R3
Connections:
- net +3V3: now also U1.11 (GPIO2)
Changed lines of the file:
@@
 $EndComp
 $Comp
-L GND #PWR8
+L GND #PWR7
 U 1 1 59932907
 P 6800 4100
-F 0 "#PWR8" H 6800 3850 50  0001 C CNN
+F 0 "#PWR7" H 6800 3850 50  0001 C CNN
 F 1 "GND" H 6800 3950 50  0000 C CNN
 F 2 "" H 6800 4100 50  0001 C CNN
@@
 $EndComp
 $Comp
-L CONN_01X01 J5
+L CONN_01X01 J2
 U 1 1 59933C1C
 P 7450 3175
-F 0 "J5" H 7450 3275 50  0000 C CNN
+F 0 "J2" H 7450 3275 50  0000 C CNN
 F 1 "CONN_01X01" V 7550 3175 50  0000 C CNN
 F 2 "mod:Alligator Pad" H 7450 3175 50  0001 C CNN
@@
 $EndComp
 $Comp
-L CONN_01X01 J6
+L CONN_01X01 J3
 U 1 1 59933C73
 P 7450 3325
-F 0 "J6" H 7450 3425 50  0000 C CNN
+F 0 "J3" H 7450 3425 50  0000 C CNN
 F 1 "CONN_01X01" V 7550 3325 50  0000 C CNN
 F 2 "mod:Alligator Pad" H 7450 3325 50  0001 C CNN
@@
 	7250 3475 7250 3700
 $Comp
-L R R4
+L R R3
 U 1 1 59935339
 P 7100 3625
-F 0 "R4" V 7180 3625 50  0000 C CNN
+F 0 "R3" V 7180 3625 50  0000 C CNN
 F 1 "10k" V 7100 3625 50  0000 C CNN
 F 2 "Resistors_SMD:R_0805_HandSoldering" V 7030 3625 50  0001 C CNN
@@
 Connection ~ 7100 3475
 $Comp
-L +3.3V #PWR13
+L +3.3V #PWR12
 U 1 1 599466C8
 P 7100 3875
-F 0 "#PWR13" H 7100 3725 50  0001 C CNN
+F 0 "#PWR12" H 7100 3725 50  0001 C CNN
 F 1 "+3.3V" H 7100 4015 50  0000 C CNN
 F 2 "" H 7100 3875 50  0001 C CNN
@@
 Wire Wire Line
 	7100 3775 7100 3875
-$Comp
-L R R3
-U 1 1 59946DA6
-P 6825 3625
-F 0 "R3" V 6905 3625 50  0000 C CNN
-F 1 "10k" V 6825 3625 50  0000 C CNN
-F 2 "Resistors_SMD:R_0805_HandSoldering" V 6755 3625 50  0001 C CNN
-F 3 "" H 6825 3625 50  0001 C CNN
-	1    6825 3625
-	0    1    1    0
-$EndComp
 Wire Wire Line
 	6625 3925 6625 4000
@@
 	6625 3775 6800 3775
 $Comp
-L +3.3V #PWR11
+L +3.3V #PWR10
 U 1 1 59948486
 P 6975 3700
-F 0 "#PWR11" H 6975 3550 50  0001 C CNN
+F 0 "#PWR10" H 6975 3550 50  0001 C CNN
 F 1 "+3.3V" H 6975 3840 50  0000 C CNN
 F 2 "" H 6975 3700 50  0001 C CNN
@@
 	4875 2525 4875 2600
 $Comp
-L GND #PWR12
+L GND #PWR11
 U 1 1 599488CC
 P 7025 1650
-F 0 "#PWR12" H 7025 1400 50  0001 C CNN
+F 0 "#PWR11" H 7025 1400 50  0001 C CNN
 F 1 "GND" H 7025 1500 50  0000 C CNN
 F 2 "" H 7025 1650 50  0001 C CNN
@@
 $EndComp
 $Comp
-L GND #PWR7
+L GND #PWR6
 U 1 1 59948924
 P 6625 4000
-F 0 "#PWR7" H 6625 3750 50  0001 C CNN
+F 0 "#PWR6" H 6625 3750 50  0001 C CNN
 F 1 "GND" H 6625 3850 50  0000 C CNN
 F 2 "" H 6625 4000 50  0001 C CNN
@@
 $EndComp
 Wire Wire Line
-	6625 3625 6675 3625
+	6625 3625 6975 3625
 Wire Wire Line
 	6975 3625 6975 3700
@@
 	5325 3925 4950 3925
 $Comp
-L GND #PWR10
+L GND #PWR9
 U 1 1 599480D5
 P 6875 2200
-F 0 "#PWR10" H 6875 1950 50  0001 C CNN
+F 0 "#PWR9" H 6875 1950 50  0001 C CNN
 F 1 "GND" H 6875 2050 50  0000 C CNN
 F 2 "" H 6875 2200 50  0001 C CNN
@@
 	6875 2200 7300 2200
 $Comp
-L +3.3V #PWR9
+L +3.3V #PWR8
 U 1 1 599481A2
 P 6850 2400
-F 0 "#PWR9" H 6850 2250 50  0001 C CNN
+F 0 "#PWR8" H 6850 2250 50  0001 C CNN
 F 1 "+3.3V" H 6850 2540 50  0000 C CNN
 F 2 "" H 6850 2400 50  0001 C CNN
@@
 F 0 "P1" H 7500 2800 50  0000 C CNN
 F 1 "CONN_01X08" V 7600 2350 50  0000 C CNN
-F 2 "" H 7500 2350 50  0000 C CNN
+F 2 "Pin_Headers:Pin_Header_Straight_1x08_Pitch2.54mm" H 7500 2350 50  0001 C CNN
 F 3 "" H 7500 2350 50  0000 C CNN
 	1    7500 2350
